Commit message: fix some errors

File: rc_description/urdf/common/laser.xacro (robot description, xacro)
@@ -32,8 +32,9 @@
     <!-- 雷达支架 -->
     <xacro:property name="support_length" value="0.1" /> <!-- 支架长度 -->
-    <xacro:property name="support_radius" value="0.01" /> <!-- 支架半径 -->
+    <xacro:property name="support_radius" value="0.35" /> <!-- 支架半径 -->
     <xacro:property name="support_x" value="0.0" /> <!-- 支架安装的x坐标 -->
     <xacro:property name="support_y" value="0.0" /> <!-- 支架安装的y坐标 -->
-    <xacro:property name="support_z" value="${ support_length / 2}" /> <!-- 支架安装的z坐标:底盘高度 / 2 + 支架高度 / 2  -->
+    <!-- <xacro:property name="support_z" value="${ support_length / 2}" />  -->
+    <xacro:property name="support_z" value="0.1" /><!-- 支架安装的z坐标:底盘高度 / 2 + 支架高度 / 2  -->
     <xacro:property name="support_m" value="0.02" /> <!-- 支架质量 -->
     <link name="support">

File: rc_description/urdf/common/radar.urdf.xacro (robot description, xacro)
@@ -44,14 +44,15 @@
                     <ray>
                         <scan>
+                        <!-- 在这里动了点手脚，把min_angle 和 max_angle改到闭合 -->
                             <horizontal>
                                 <samples>360</samples>
                                 <resolution>1</resolution>
-                                <min_angle>-2.35619445</min_angle>
-                                <max_angle>2.35619445</max_angle>
+                                <min_angle>-3.1415926</min_angle>
+                                <max_angle>3.1415926</max_angle>
                             </horizontal>
                         </scan>
                         <range>
-                            <min>0.260</min>
-                            <max>7.5</max>
+                            <min>0.05</min>
+                            <max>10.0</max>
                             <resolution>0.015</resolution>
                         </range>
@@ -62,8 +63,10 @@
                         </noise>
                     </ray>
+                    <!-- 这里也做了手脚，做了命名空间的传入，让其可以支持多辆车都装载雷达并且发布话题到各自命名空间下 -->
+                    <!-- 否则不同车会发布雷达数据到同一个话题/scan下 -->
                     <plugin name="gazebo_rplidar" filename="libgazebo_ros_laser.so">
-                        <robotNamespace>/</robotNamespace>
-                        <topicName>/scan</topicName>
-                        <frameName>radar_link</frameName>
+                        <robotNamespace>$(arg robot_namespace)</robotNamespace>
+                        <topicName>scan</topicName>
+                        <frameName>$(arg robot_namespace)/radar_link</frameName>
                     </plugin>
                 </sensor>

File: rc_description/urdf/rabbit/rabbit.urdf.xacro (robot description, xacro)
@@ -7,17 +7,46 @@
     <xacro:arg name="robot_namespace" default="robot1" />
     <xacro:arg name="use_sim" default="true"/>
+    <xacro:arg name="load_cube" default="true" />
     <xacro:include filename="$(find rc_description)/urdf/rabbit/chassis.urdf.xacro"/>
     <xacro:chassis roller_type="$(arg roller_type)" robot_namespace="$(arg robot_namespace)"/>
-    <!-- <xacro:if value="$(arg load_radar)">
+    <xacro:if value="$(arg load_radar)">
         <xacro:include filename="$(find rc_description)/urdf/common/radar.urdf.xacro"/>
         <xacro:RADAR connected_to="base_link" radar_name="radar" use_sim="$(arg use_sim)"
-                     xyz="0.23897 0 0.057"
+                     xyz="0.0 0 0.1"
                      rpy="0.0 0.0 0.0"/>
-    </xacro:if> -->
+    </xacro:if>
     <xacro:if value="$(arg load_action)">
         <xacro:include filename="$(find rc_description)/urdf/common/action.urdf.xacro"/>
         <xacro:ACTION connected_to="base_link" action_name="location_action" use_sim="$(arg use_sim)" robot_namespace="$(arg robot_namespace)"
-                      xyz="-0.035 0 -0.06"
+                      xyz="0.0 0 -0.06"
                       rpy="0.0 0.0 0.0"/>
+    </xacro:if>
+    <xacro:if value="$(arg load_cube)">
+        <!-- 添加圆柱体到机器人上，以便laser可以检测到 -->
+        <link name="cylinder_link">
+            <visual>
+                <geometry>
+                    <cylinder radius="0.28" length="0.1"/> <!-- 圆柱体的视觉尺寸 -->
+                </geometry>
+                <material name="red">
+                    <color rgba="1 0 0 1"/> <!-- 红色 -->
+                </material>
+            </visual>
+            <collision>
+                <geometry>
+                    <cylinder radius="0.28" length="0.1"/> <!-- 圆柱体的碰撞尺寸 -->
+                </geometry>
+            </collision>
+            <inertial>
+                <mass value="1.0"/> <!-- 质量 -->
+                <origin xyz="0 0 0" rpy="0 0 0"/>
+                <inertia ixx="0.001" ixy="0.0" ixz="0.0" iyy="0.001" iyz="0.0" izz="0.001"/>
+            </inertial>
+        </link>
+        <joint name="cylinder_joint" type="fixed">
+            <parent link="base_link"/>
+            <child link="cylinder_link"/>
+            <origin xyz="0.0 0 0.10" rpy="0 0 0"/> <!-- 圆柱体相对于 base_link 的位置 -->
+        </joint>
     </xacro:if>
     <gazebo>

File: rc_description/urdf/rc_r2/chassis.urdf.xacro (robot description, xacro)
@@ -5,5 +5,5 @@
     <xacro:include filename="$(find rc_description)/urdf/rc_r2/omni_wheel.urdf.xacro"/>
     <xacro:include filename="$(find rc_description)/urdf/common/action.urdf.xacro" />
-    <!-- <xacro:include filename="$(find urdf01_gazebo)/urdf/omni_chassis/laseer_sensor.xacro" /> -->
+    <xacro:include filename="$(find rc_description)/urdf/common/laser.xacro" />
     <xacro:property name="roller_type" value="simple" />
     <!-- https://upload.wikimedia.org/wikipedia/commons/5/52/Wheelbase_and_Track.png -->
@@ -63,5 +63,5 @@
     </link>
     <xacro:ACTION connected_to="base_link" action_name="location_action" use_sim="$(arg use_sim)" robot_namespace="$(arg robot_namespace)"
-                      xyz="-0.035 0 0"
+                      xyz="0.0 0 0"
                       rpy="0.0 0.0 0.0"
                       />
